File: active-drag-system-pcb/active-drag-system-pcb.kicad_sch (KiCad schematic)
At the start: 58 parts, among them J1 Conn_01x02_Socket, J1 USB_B_Micro, SW1 PTS815 SJM 250 SMTR LFS, U1 TPS51386RJNR, U2 LD39200PU33R, U3 PMEG3050EP_115, U4 PMEG3050EP_115, U5 RP2040, U6 W25Q128JVS, Y1 ABM8-272-T3

Commit message: Literally everything has footprints and is pretty connected together on schematic except for IIM
Parts:
- removed L1: 1.5uH, symbol Device:L
- removed Y1: ABM8-272-T3, Crystal:Crystal_SMD_3225-4Pin_3.2x2.5mm, symbol Device:Crystal_GND24
- added C46: 1000pF, Capacitor_SMD:C_0402_1005Metric_Pad0.74x0.62mm_HandSolder, symbol Device:C
- added C47, C48, C49, C50, C51: 100n, Capacitor_SMD:C_0201_0603Metric_Pad0.64x0.40mm_HandSolder, symbol Device:C
- added L1: 104CDMCCDS-1R5MC, IND_-1R5MC_SUM, symbol 104CDMCCDS-1R5MC:104CDMCCDS-1R5MC
- added Q7: DMG1012T, Package_TO_SOT_SMD:SOT-523, symbol Transistor_FET:DMG1012T
- added U13: MS5611-01BA, Package_LGA:LGA-8_3x5mm_P1.25mm, symbol Sensor_Pressure:MS5611-01BA
- added U14: LSM6DSV16XTR, LGA14L_LSM6_STM, symbol 2024-09-29_14-58-49:LSM6DSV16XTR
- added U15: ADXL375BCCZ, LGA_CC-14-1_ADI, symbol 2024-09-29_15-03-30:ADXL375BCCZ
- added U16: IIM-42653, IIM-42653:PQFN50P250X300X97-14N, symbol IIM-42653:IIM-42653
- added X1: ABM8-272-T3, ABM8-272-T3_ABR, symbol ABM8-272-T3:ABM8-272-T3
- C1, C5: footprint (none) -> Capacitor_SMD:C_0201_0603Metric_Pad0.64x0.40mm_HandSolder; Dielectric (none) -> X5R; Max Voltage (none) -> 16 V; Tolerance (none) -> 10%
- C10, C7, C8, C9: footprint (none) -> Capacitor_SMD:C_0402_1005Metric_Pad0.74x0.62mm_HandSolder; Dielectric (none) -> X5R; Max Voltage (none) -> 10V; Tolerance (none) -> 20%
- C11, C12, C2, C3: footprint (none) -> Capacitor_SMD:C_0805_2012Metric_Pad1.18x1.45mm_HandSolder; Dielectric (none) -> X5R; Max Voltage (none) -> 16V; Tolerance (none) -> 10%
- C13: value 2.2uF -> 2.2u; footprint Capacitor_SMD:C_0402_1005Metric -> Capacitor_SMD:C_0402_1005Metric_Pad0.74x0.62mm_HandSolder; Dielectric (none) -> X5R; Max Voltage (none) -> 6.3V; Tolerance (none) -> 20%
- C14, C15, C19, C20, C21, C22, C23, C24, C27: footprint (none) -> Capacitor_SMD:C_0201_0603Metric_Pad0.64x0.40mm_HandSolder; Dielectric (none) -> X5R; Max Voltage (none) -> 6.3V; Tolerance (none) -> 10%
- C16, C17, C18: value 2.2uF -> 2.2u; footprint (none) -> Capacitor_SMD:C_0402_1005Metric_Pad0.74x0.62mm_HandSolder; Dielectric (none) -> X5R; Max Voltage (none) -> 6.3V; Tolerance (none) -> 20%
- C25, C26: footprint (none) -> Capacitor_SMD:C_0201_0603Metric; Dielectric (none) -> C0G; Max Voltage (none) -> 25V; Tolerance (none) -> 5%
- C4: footprint (none) -> Capacitor_SMD:C_0402_1005Metric_Pad0.74x0.62mm_HandSolder; Dielectric (none) -> X5R; Max Voltage (none) -> 6.3V; Tolerance (none) -> 20%
- C6: value 22pF -> 22p; footprint (none) -> Capacitor_SMD:C_0201_0603Metric; Dielectric (none) -> C0G; Max Voltage (none) -> 25V; Tolerance (none) -> 5%
- R1: value 560k -> 100k; footprint (none) -> Resistor_SMD:R_0402_1005Metric_Pad0.72x0.64mm_HandSolder; Power (none) -> 1/16W; Tolerance (none) -> 0.1%
- R2: value 80k -> 100k; footprint (none) -> Resistor_SMD:R_0402_1005Metric_Pad0.72x0.64mm_HandSolder; Power (none) -> 1/16W; Tolerance (none) -> 0.1%
- R28, R29: footprint (none) -> Resistor_SMD:R_0201_0603Metric_Pad0.64x0.40mm_HandSolder; Power (none) -> 50mW; Tolerance (none) -> 1%
- R3, R5, R7: footprint (none) -> Resistor_SMD:R_0402_1005Metric_Pad0.72x0.64mm_HandSolder; Power (none) -> 1/16W; Tolerance (none) -> 0.1%
- R30, R32, R33, R9: footprint (none) -> Resistor_SMD:R_0402_1005Metric_Pad0.72x0.64mm_HandSolder; Power (none) -> 63mW; Tolerance (none) -> 1%
- R31: footprint (none) -> Resistor_SMD:R_0603_1608Metric_Pad0.98x0.95mm_HandSolder; Power (none) -> 100mW; Tolerance (none) -> 1%
- R4: value 0 -> 200k; footprint (none) -> Resistor_SMD:R_0402_1005Metric_Pad0.72x0.64mm_HandSolder; Power (none) -> 63mW; Tolerance (none) -> 1%
- R6: value 0 -> 100k; footprint (none) -> Resistor_SMD:R_0402_1005Metric_Pad0.72x0.64mm_HandSolder; Power (none) -> 63mW; Tolerance (none) -> 1%
Connections:
- net +1V1: now also C15.1, C17.1; no longer C14.1, C16.1
- net +3V3: now also C14.1, C16.1, C47.1, C48.1, C49.1, C50.1, C51.1, Q7.1 (G), U13.1 (VDD), U13.2 (PS), U14.12 (CS), U14.5 (VDD_IO), U14.8 (VDD), U15.1 (VDD_I/O), U15.12 (SDO/ALT_ADDRESS), U15.6 (VS), U15.7 (*CS); no longer C15.1, C17.1
- net +5V: now also L1.1
- net -BATT: now also R6.2, R7.1, C46.2, C47.2, C48.2, C49.2, C50.2, C51.2, U13.3 (GND), U13.4 (CSB), U13.5 (CSB), U14.1 (SDO/SA0), U14.2 (SDx/AH1/QVAR1), U14.3 (SCx/AH2/QVAR2), U14.6 (GND), U14.7 (GND), U15.11 (RESERVED), U15.2 (GND), U15.3 (RESERVED), U15.4 (GND), U15.5 (GND), X1.2, X1.4; no longer R7.2
- net GPIO25: now also R9.1; no longer R9.2
- net GPIO29_ADC3: now also Q7.2 (S)
- net XIN: now also X1.1
- net at U1.8 (VBST): now also C5.2; no longer R4.1
- net at R4.2: now also R6.1, C46.1, Q7.3 (D); no longer C5.1
- net VSYS: now reaches C11.1, R8.1, U2.6 (IN), U3.1 (K), U4.1 (K)
- net VSYS: now also R4.1
- net at C25.1, R32.2: now also X1.3
- net at R5.1, U1.4 (FB): now also C6.1, R7.2; no longer R6.1, R7.1
- net at U1.7 (SW): now also C5.1, L1.2; no longer C5.2
- net at D7.2: now also R9.2; no longer R9.1
- net GPIO0 renamed I2C0_SDA
- net I2C0_SDA: now also U13.7 (SDI/SDA), U14.14 (SDA), U15.13 (SDA/SDI/SDIO)
- net GPIO1 renamed I2C0_SCL
- net I2C0_SCL: now also U13.8 (SCLK), U14.13 (SCL), U15.14 (SCL/SCLK)
- new net HIGHG_INT1: U15.8 (INT1)
- new net HIGHG_INT2: U15.9 (INT2)
- new net LOWG_INT1: U14.4 (INT1), U14.9 (INT2)
Other:
- note added: "Altimeter"
- note added: "High-G IMU"
- note added: "Low-G IMU"
- note added: "This one's crazy"
- moved on the sheet: C7, R8, U2, U3, U4

Commit message: Populated IIM-42653
Parts:
- added C52: 10nF, symbol Device:C
- added C53: 100nF, symbol Device:C
- added C54: 2200nF, symbol Device:C
- added R34: 10k, Resistor_SMD:R_0201_0603Metric_Pad0.64x0.40mm_HandSolder, symbol Device:R
- added R35: 10k, symbol Device:R
Connections:
- net +3V3: now also U16.12 (AP_CS), U16.5 (VDDIO), U16.8 (VDD), C52.1, C53.1, C54.1, R34.2, R35.1
- net -BATT: now also U16.1 (AP_SDO/AP_AD0), U16.10 (AUX1_CS), U16.11 (AUX1_SDO), U16.2 (AUX1_SDIO), U16.3 (AUX1_SCLK), U16.6 (GND), U16.7 (RESV), C52.2, C53.2, C54.2
- net GPIO21: now also U16.9 (INT2/FSYNC/CLKIN)
- net I2C0_SCL: now also U16.13 (AP_SCL/AP_SCLK), R34.1
- net I2C0_SDA: now also U16.14 (AP_SDA/AP_SDIO/AP_SDI), R35.2
- net MIDG_INT1: now reaches U16.4 (INT1/INT)
Other:
- note added: "I2C0 Pullups"
